File: pcb/NumPad/led_matrix.sch (KiCad schematic (older format))
At the start: 20 parts

Commit message: started Numpad Layout
Parts:
- D21, D22, D23, D24, D25, D26, D27, D28, D29, D30, D31, D32, D33, D34, D35, D36, D37, D38, D39, D40: footprint footprints:LED_3MM -> footprints:CHERRY_MX_LED
Changed lines of the file:
@@
 F 0 "D21" H 2200 1750 50  0000 C CNN
 F 1 "L_+" H 2200 1550 50  0000 C CNN
-F 2 "footprints:LED_3MM" H 2200 1650 50  0001 C CNN
+F 2 "footprints:CHERRY_MX_LED" H 2200 1650 50  0001 C CNN
 F 3 "" H 2200 1650 50  0001 C CNN
 	1    2200 1650
@@
 F 0 "D26" H 2600 1750 50  0000 C CNN
 F 1 "L_-" H 2600 1550 50  0000 C CNN
-F 2 "footprints:LED_3MM" H 2600 1650 50  0001 C CNN
+F 2 "footprints:CHERRY_MX_LED" H 2600 1650 50  0001 C CNN
 F 3 "" H 2600 1650 50  0001 C CNN
 	1    2600 1650
@@
 F 0 "D31" H 3000 1750 50  0000 C CNN
 F 1 "L_*" H 3000 1550 50  0000 C CNN
-F 2 "footprints:LED_3MM" H 3000 1650 50  0001 C CNN
+F 2 "footprints:CHERRY_MX_LED" H 3000 1650 50  0001 C CNN
 F 3 "" H 3000 1650 50  0001 C CNN
 	1    3000 1650
@@
 F 0 "D36" H 3400 1750 50  0000 C CNN
 F 1 "L_/" H 3400 1550 50  0000 C CNN
-F 2 "footprints:LED_3MM" H 3400 1650 50  0001 C CNN
+F 2 "footprints:CHERRY_MX_LED" H 3400 1650 50  0001 C CNN
 F 3 "" H 3400 1650 50  0001 C CNN
 	1    3400 1650
@@
 F 0 "D22" H 2200 2350 50  0000 C CNN
 F 1 "L_7" H 2200 2150 50  0000 C CNN
-F 2 "footprints:LED_3MM" H 2200 2250 50  0001 C CNN
+F 2 "footprints:CHERRY_MX_LED" H 2200 2250 50  0001 C CNN
 F 3 "" H 2200 2250 50  0001 C CNN
 	1    2200 2250
@@
 F 0 "D27" H 2600 2350 50  0000 C CNN
 F 1 "L_8" H 2600 2150 50  0000 C CNN
-F 2 "footprints:LED_3MM" H 2600 2250 50  0001 C CNN
+F 2 "footprints:CHERRY_MX_LED" H 2600 2250 50  0001 C CNN
 F 3 "" H 2600 2250 50  0001 C CNN
 	1    2600 2250
@@
 F 0 "D32" H 3000 2350 50  0000 C CNN
 F 1 "L_9" H 3000 2150 50  0000 C CNN
-F 2 "footprints:LED_3MM" H 3000 2250 50  0001 C CNN
+F 2 "footprints:CHERRY_MX_LED" H 3000 2250 50  0001 C CNN
 F 3 "" H 3000 2250 50  0001 C CNN
 	1    3000 2250
@@
 F 0 "D37" H 3400 2350 50  0000 C CNN
 F 1 "L_FN2" H 3400 2150 50  0000 C CNN
-F 2 "footprints:LED_3MM" H 3400 2250 50  0001 C CNN
+F 2 "footprints:CHERRY_MX_LED" H 3400 2250 50  0001 C CNN
 F 3 "" H 3400 2250 50  0001 C CNN
 	1    3400 2250
@@
 F 0 "D23" H 2200 2950 50  0000 C CNN
 F 1 "L_4" H 2200 2750 50  0000 C CNN
-F 2 "footprints:LED_3MM" H 2200 2850 50  0001 C CNN
+F 2 "footprints:CHERRY_MX_LED" H 2200 2850 50  0001 C CNN
 F 3 "" H 2200 2850 50  0001 C CNN
 	1    2200 2850
@@
 F 0 "D28" H 2600 2950 50  0000 C CNN
 F 1 "L_5" H 2600 2750 50  0000 C CNN
-F 2 "footprints:LED_3MM" H 2600 2850 50  0001 C CNN
+F 2 "footprints:CHERRY_MX_LED" H 2600 2850 50  0001 C CNN
 F 3 "" H 2600 2850 50  0001 C CNN
 	1    2600 2850
@@
 F 0 "D33" H 3000 2950 50  0000 C CNN
 F 1 "L_6" H 3000 2750 50  0000 C CNN
-F 2 "footprints:LED_3MM" H 3000 2850 50  0001 C CNN
+F 2 "footprints:CHERRY_MX_LED" H 3000 2850 50  0001 C CNN
 F 3 "" H 3000 2850 50  0001 C CNN
 	1    3000 2850
@@
 F 0 "D38" H 3400 2950 50  0000 C CNN
 F 1 "L_FN1" H 3400 2750 50  0000 C CNN
-F 2 "footprints:LED_3MM" H 3400 2850 50  0001 C CNN
+F 2 "footprints:CHERRY_MX_LED" H 3400 2850 50  0001 C CNN
 F 3 "" H 3400 2850 50  0001 C CNN
 	1    3400 2850
@@
 F 0 "D24" H 2200 3550 50  0000 C CNN
 F 1 "L_1" H 2200 3350 50  0000 C CNN
-F 2 "footprints:LED_3MM" H 2200 3450 50  0001 C CNN
+F 2 "footprints:CHERRY_MX_LED" H 2200 3450 50  0001 C CNN
 F 3 "" H 2200 3450 50  0001 C CNN
 	1    2200 3450
@@
 F 0 "D34" H 3000 3550 50  0000 C CNN
 F 1 "L_3" H 3000 3350 50  0000 C CNN
-F 2 "footprints:LED_3MM" H 3000 3450 50  0001 C CNN
+F 2 "footprints:CHERRY_MX_LED" H 3000 3450 50  0001 C CNN
 F 3 "" H 3000 3450 50  0001 C CNN
 	1    3000 3450
@@
 F 0 "D39" H 3400 3550 50  0000 C CNN
 F 1 "L_=" H 3400 3350 50  0000 C CNN
-F 2 "footprints:LED_3MM" H 3400 3450 50  0001 C CNN
+F 2 "footprints:CHERRY_MX_LED" H 3400 3450 50  0001 C CNN
 F 3 "" H 3400 3450 50  0001 C CNN
 	1    3400 3450
@@
 F 0 "D25" H 2200 4150 50  0000 C CNN
 F 1 "L_0" H 2200 3950 50  0000 C CNN
-F 2 "footprints:LED_3MM" H 2200 4050 50  0001 C CNN
+F 2 "footprints:CHERRY_MX_LED" H 2200 4050 50  0001 C CNN
 F 3 "" H 2200 4050 50  0001 C CNN
 	1    2200 4050
@@
 F 0 "D30" H 2600 4150 50  0000 C CNN
 F 1 "L_," H 2600 3950 50  0000 C CNN
-F 2 "footprints:LED_3MM" H 2600 4050 50  0001 C CNN
+F 2 "footprints:CHERRY_MX_LED" H 2600 4050 50  0001 C CNN
 F 3 "" H 2600 4050 50  0001 C CNN
 	1    2600 4050
@@
 F 0 "D35" H 3000 4150 50  0000 C CNN
 F 1 "L_." H 3000 3950 50  0000 C CNN
-F 2 "footprints:LED_3MM" H 3000 4050 50  0001 C CNN
+F 2 "footprints:CHERRY_MX_LED" H 3000 4050 50  0001 C CNN
 F 3 "" H 3000 4050 50  0001 C CNN
 	1    3000 4050
@@
 F 0 "D40" H 3400 4150 50  0000 C CNN
 F 1 "L_FN0" H 3400 3950 50  0000 C CNN
-F 2 "footprints:LED_3MM" H 3400 4050 50  0001 C CNN
+F 2 "footprints:CHERRY_MX_LED" H 3400 4050 50  0001 C CNN
 F 3 "" H 3400 4050 50  0001 C CNN
 	1    3400 4050
@@
 F 0 "D29" H 2600 3550 50  0000 C CNN
 F 1 "L_2" H 2600 3350 50  0000 C CNN
-F 2 "footprints:LED_3MM" H 2600 3450 50  0001 C CNN
+F 2 "footprints:CHERRY_MX_LED" H 2600 3450 50  0001 C CNN
 F 3 "" H 2600 3450 50  0001 C CNN
 	1    2600 3450
